Commit message: 모터 링크 추가 및 tf 시각화 옵션 수정

File: urdf/car.urdf (robot description, URDF)
Before this commit: robot car, 1 links, 0 joints
Links:
- added link left_motor; visual mesh filename=package://awesome_driver/meshes/rear_actuator.stl
Joints:
- added joint left_motor_mnt: type fixed, parent base_link, child left_motor, origin xyz=0 0.0556 0.0195 rpy=0 0 0

Commit message: 좌측 바퀴 추가 및 축 정렬

File: urdf/car.urdf (robot description, URDF)
Before this commit: robot car, 2 links, 1 joints
Links:
- added link left_wheel; visual mesh filename=package://awesome_driver/meshes/left_rear_wheel.stl
Joints:
- added joint left_motor_wheel: type continuous, parent left_motor, child left_wheel, origin xyz=0 0.0264 -0.007 rpy=0 0 0, axis 0 1 0

Commit message: 볼 캐스터 추가

File: urdf/car.urdf (robot description, URDF)
Before this commit: robot car, 3 links, 2 joints
Links:
- added link caster; visual sphere radius=0.01
Joints:
- added joint caster_joint: type fixed, parent base_link, child caster, origin xyz=0.28 0 0 rpy=0 0 0

Commit message: 메인 프레임에 재질 적용

File: urdf/car.urdf (robot description, URDF)
Before this commit: robot car, 4 links, 3 joints
Links:
- link base_link: geometry visual mesh filename=package://awesome_driver/meshes/main_frame.obj

Commit message: 바퀴 콜리전 추가

File: urdf/car.urdf (robot description, URDF)
Before this commit: robot car, 4 links, 3 joints
Links:
- link left_wheel: geometry collision cylinder length=0.0265 radius=0.03448; visual mesh filename=package://awesome_driver/meshes/left_rear_wheel.stl

Commit message: 볼 캐스터 콜리전 추가 및 시각화 옵션 수정

File: urdf/car.urdf (robot description, URDF)
Before this commit: robot car, 4 links, 3 joints
Links:
- link caster: geometry collision sphere radius=0.01; visual sphere radius=0.01

Commit message: macro 기반 좌측 및 우측 시스템 생성

File: urdf/car.urdf (robot description, URDF)
Before this commit: robot car, 4 links, 3 joints
Links:
- added link right_motor; visual mesh filename=package://awesome_driver/meshes/rear_actuator.stl
- added link right_wheel; collision cylinder length=0.0265 radius=0.03448; visual mesh filename=package://awesome_driver/meshes/left_rear_wheel.stl
Joints:
- added joint right_motor_mnt: type fixed, parent base_link, child right_motor, origin xyz=0 -0.0556 0.0195 rpy=0 0 3.14159265359
- added joint right_motor_wheel: type continuous, parent right_motor, child right_wheel, origin xyz=0 0.0264 -0.007 rpy=0 0 0, axis 0 1 0

File: urdf/car.xacro (robot description, xacro)
@@ -65,3 +65,5 @@
         </joint>
     </xacro:macro>
+    <xacro:rear_system prefix="left" y_offset="0.0556" yaw="0"/>
+    <xacro:rear_system prefix="right" y_offset="-0.0556" yaw="${pi}"/>
 </robot>
