Commit message: macro 정의 및 기본 구조 작성

File: urdf/car.xacro (robot description, xacro)
@@ -26,4 +26,14 @@
         </collision>
     </link>
+    <xacro:macro name="rear_system" params="prefix y_offset yaw">
+        <link name="${prefix}_motor">
+        </link>
+        <link name="${prefix}_wheel">
+        </link>
+        <joint name="${prefix}_motor_mnt" type="fixed">
+        </joint>
+        <joint name="${prefix}_motor_wheel" type="continuous">
+        </joint>
+    </xacro:macro>
     <link name="left_motor">
         <visual>

Commit message: macro 세부 내용 기입

File: urdf/car.xacro (robot description, xacro)
@@ -28,48 +28,40 @@
     <xacro:macro name="rear_system" params="prefix y_offset yaw">
         <link name="${prefix}_motor">
+            <visual>
+                <geometry>
+                    <mesh filename="package://awesome_driver/meshes/rear_actuator.stl"/>
+                </geometry>
+                <material name="gray">
+                    <color rgba="0.8 0.8 0.8 1"/>
+                </material>
+            </visual>
         </link>
         <link name="${prefix}_wheel">
+            <visual>
+                <geometry>
+                    <mesh filename="package://awesome_driver/meshes/left_rear_wheel.stl"/>
+                </geometry>
+                <material name="black">
+                    <color rgba="0.2 0.2 0.2 1"/>
+                </material>
+            </visual>
+            <collision>
+                <geometry>
+                    <cylinder radius="0.03448" length="0.0265"/>
+                </geometry>
+                <origin xyz="0 0 0" rpy="${pi/2} 0 0"/>
+            </collision>
         </link>
         <joint name="${prefix}_motor_mnt" type="fixed">
+            <parent link="base_link"/>
+            <child link="${prefix}_motor"/>
+            <origin xyz="0 ${y_offset} 0.0195" rpy="0 0 ${yaw}"/>
         </joint>
         <joint name="${prefix}_motor_wheel" type="continuous">
+            <parent link="${prefix}_motor"/>
+            <child link="${prefix}_wheel"/>
+            <axis xyz="0 1 0"/>
+            <origin xyz="0 0.0264 -0.007" rpy="0 0 0"/>
         </joint>
     </xacro:macro>
-    <link name="left_motor">
-        <visual>
-            <geometry>
-                <mesh filename="package://awesome_driver/meshes/rear_actuator.stl"/>
-            </geometry>
-            <material name="gray">
-                <color rgba="0.8 0.8 0.8 1"/>
-            </material>
-        </visual>
-    </link>
-    <joint name="left_motor_mnt" type="fixed">
-        <parent link="base_link"/>
-        <child link="left_motor"/>
-        <origin xyz="0 0.0556 0.0195" rpy="0 0 0"/>
-    </joint>
-    <link name="left_wheel">
-        <visual>
-            <geometry>
-                <mesh filename="package://awesome_driver/meshes/left_rear_wheel.stl"/>
-            </geometry>
-            <material name="black">
-                <color rgba="0.2 0.2 0.2 1"/>
-            </material>
-        </visual>
-        <collision>
-            <geometry>
-                <cylinder radius="0.03448" length="0.0265"/>
-            </geometry>
-            <origin xyz="0 0 0" rpy="${pi/2} 0 0"/>
-        </collision>
-    </link>
-    <joint name="left_motor_wheel" type="continuous">
-        <parent link="left_motor"/>
-        <child link="left_wheel"/>
-        <axis xyz="0 1 0"/>
-        <origin xyz="0 0.0264 -0.007" rpy="0 0 0"/>
-    </joint>
 </robot>

Commit message: gazebo element를 통한 재질 반영 및 위치 수정

File: urdf/car.xacro (robot description, xacro)
@@ -11,4 +11,7 @@
         <xacro:inertial_base/>
     </link>
+    <gazebo reference="base_link">
+        <pose>0 0 0.3 0 0 0</pose>
+    </gazebo>
     <joint name="caster_joint" type="fixed">
         <parent link="base_link"/>
@@ -29,4 +32,7 @@
         <xacro:inertial_caster/>
     </link>
+    <gazebo reference="caster">
+        <material>Gazebo/RedBright</material>
+    </gazebo>
     <xacro:macro name="rear_system" params="prefix y_offset yaw">
         <link name="${prefix}_motor">
@@ -69,4 +75,10 @@
             <origin xyz="0 0.0264 -0.007" rpy="0 0 0"/>
         </joint>
+        <gazebo reference="${prefix}_motor">
+            <material>Gazebo/Gold</material>
+        </gazebo>
+        <gazebo reference="${prefix}_wheel">
+            <material>Gazebo/Grey</material>
+        </gazebo>
     </xacro:macro>
     <xacro:rear_system prefix="left" y_offset="0.0556" yaw="0"/>

Commit message: gazebo_ros_control plugin 및 transmission element 추가, gazebo_car.launch 파일 수정 및 gazebo_control.launch 파일 추가

File: urdf/car.xacro (robot description, xacro)
@@ -91,6 +91,21 @@
             <material>Gazebo/Grey</material>
         </gazebo>
+        <transmission name="${prefix}_transmission">
+            <type>transmission_interface/SimpleTransmission</type>
+            <joint name="${prefix}_motor_wheel">
+                <hardwareInterface>hardware_interface/EffortJointInterface</hardwareInterface>
+            </joint>
+            <actuator name="${prefix}_actuator">
+                <mechanicalReduction>1</mechanicalReduction>
+            </actuator>
+        </transmission>
     </xacro:macro>
     <xacro:rear_system prefix="left" y_offset="0.0556" yaw="0"/>
     <xacro:rear_system prefix="right" y_offset="-0.0556" yaw="${pi}"/>
+    <gazebo>
+        <plugin name="gazebo_ros_control" filename="libgazebo_ros_control.so">
+            <robotNamespace>/car</robotNamespace>
+            <robotSimType>gazebo_ros_control/DefaultRobotHWSim</robotSimType>
+        </plugin>
+    </gazebo>
 </robot>
